File: pi-crust.sch (EAGLE design)
At the start: 11 parts

Commit message: Replaced 5V pins in ports to 3V3. Added 2 ports level converter for convert data lines from 3V3 to 5V. Updated labeling of pins for both revisions of RPi...
Parts:
- added JP11: (no value), pinhead:PINHD-1X2
- added LOGO1: OSHW_LOGO_8MILX0100-NT, ohw-logo:OSHW_LOGO_8MILX0100-NT
- added Q1, Q2: (no value), #_GM99:BSS138SMD
- added R1, R2, R3, R4: (no value), rcl:R-EU_R0603
- JP3: value 5V -> (none); device pinhead:PINHD-1X3 -> pinhead:PINHD-1X4
- JP6: value UART -> (none); device pinhead:PINHD-1X4 -> pinhead:PINHD-1X3
Connections:
- new net N$1: JP11.2, Q2.S, R2.1
- new net N$2: JP4.2, Q2.D, R4.1
- new net N$3: JP11.1, Q1.S, R1.1
- new net N$4: JP4.1, Q1.D, R3.1
- net 3V3: now also JP10.2, JP7.2, JP8.2, JP9.2, Q1.G, Q2.G, R1.2, R2.2; no longer JP4.1, JP4.2
- net 5V: now also JP3.4, R3.2, R4.2; no longer JP10.2, JP6.2, JP7.2, JP8.2, JP9.2
- net UART_RX: now also JP6.3; no longer JP6.4
- net UART_TX: now also JP6.2; no longer JP6.3
Other:
- moved on the sheet: JP4
