File: pi-crust.brd (EAGLE design)
At the start: 43.7 x 40.4 mm, 11 parts

Commit message: Replaced 5V pins in ports to 3V3. Added 2 ports level converter for convert data lines from 3V3 to 5V. Updated labeling of pins for both revisions of RPi...
Parts:
- added JP11: (no value), pinhead:1X02
- added LOGO1: OSHW_LOGO_8MILX0100-NT, ohw-logo:OSHW_8X100_NOTEXT
- added Q1, Q2: (no value), #_GM99:SOT23
- added R1, R2, R3, R4: (no value), rcl:R0603
- JP3: value 5V -> (none); device pinhead:1X03 -> pinhead:1X04
- JP6: value UART -> (none); device pinhead:1X04 -> pinhead:1X03
- moved JP4 5.36 mm to (11.7, 37.6), turned to 270 degrees
- moved JP6 1.27 mm to (17.8, 38.1)
- moved JP3 0.28 mm to (40.4, 7.49)
Connections:
- new net N$1: JP11.2, Q2.1, R2.1
- new net N$2: JP4.2, Q2.3, R4.1
- new net N$3: JP11.1, Q1.1, R1.1
- new net N$4: JP4.1, Q1.3, R3.1
- net 3V3: now also JP10.2, JP7.2, JP8.2, JP9.2, Q1.2, Q2.2, R1.2, R2.2; no longer JP4.1, JP4.2
- net 5V: now also JP3.4, R3.2, R4.2; no longer JP10.2, JP6.2, JP7.2, JP8.2, JP9.2
- net UART_RX: now also JP6.3; no longer JP6.4
- net UART_TX: now also JP6.2; no longer JP6.3
Routing:
- net 3V3: track 42.3 -> 81.0 mm, vias 0 -> 3
- net 5V: track 109.4 -> 87.0 mm, vias 0 -> 2
- net N$4: track 0.00 -> 13.7 mm
- net N$2: track 0.00 -> 7.86 mm
- net N$1: track 0.00 -> 6.62 mm
- net N$3: track 0.00 -> 6.57 mm
- net SPI_MOSI: track 27.8 -> 28.4 mm
- net GND: track 88.7 -> 88.2 mm
Other:
- board text added: "21/27"
- board text added: "3V3 MAX."
- board text added: "ALL PORTS"
- board text added: "GPCLK0"
- board text added: "LEVEL"
- board text added: "Pi Crust v6"
- board text added: "R1/R2"
- board text added: "UART"
- board text added: "by @joewalnes @hamshop.cz (CC-SA)"
- board text added: "picru.st"
- board text removed: "21"
- board text removed: "Pi Crust v5"
- board text removed: "by @joewalnes (CC-SA)"
- board text removed: "picru.st/"

Commit message: Minor changes..
Routing:
- net 3V3: track 81.0 -> 80.7 mm, vias 3 -> 2
Changed lines of the file:
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@@
 <wire x1="8.343" y1="38.1" x2="8.382" y2="38.735" width="0.1524" layer="1"/>
 <wire x1="25.4" y1="21.59" x2="25.654" y2="21.59" width="0.1524" layer="1"/>
-<wire x1="25.654" y1="21.59" x2="25.654" y2="22.352" width="0.1524" layer="1"/>
-<via x="25.654" y="22.352" extent="1-16" drill="0.6"/>
-<wire x1="25.654" y1="22.352" x2="25.4" y2="22.352" width="0.1524" layer="16"/>
 <wire x1="25.4" y1="22.352" x2="25.4" y2="26.67" width="0.1524" layer="16"/>
 <wire x1="20.32" y1="2.54" x2="20.32" y2="1.016" width="0.1524" layer="16"/>
@@
 <wire x1="25.019" y1="24.892" x2="25.4" y2="25.273" width="0.1524" layer="1"/>
 <wire x1="25.4" y1="25.273" x2="25.4" y2="26.67" width="0.1524" layer="1"/>
+<wire x1="25.4" y1="22.352" x2="25.4" y2="21.59" width="0.4064" layer="16"/>
 <wire x1="6.604" y1="36.8046" x2="6.858" y2="36.8554" width="0" layer="19" extent="1-16"/>
 </signal>
